File: freezepad-pcb.kicad_pcb (KiCad board)
At the start: 2 copper layers, 74 x 87 mm, 24 parts

Commit message: Added Routing
Routing:
- net GND: track 9.76 -> 5.50 mm, vias 0 -> 2
- added copper zone on B.Cu, net GND
- added copper zone on F.Cu, net GND
Changed lines of the file:
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@@
 	)
 	(segment
-		(start 59.4673 -56.8027)
-		(end 61.65 -54.62)
+		(start 28.5 -54.5)
+		(end 23 -54.5)
 		(width 0.2)
 		(layer "F.Cu")
 		(net 2)
 	)
-	(segment
-		(start 54.4573 -56.8027)
-		(end 59.4673 -56.8027)
-		(width 0.2)
-		(layer "F.Cu")
+	(via
+		(at 23 -54.5)
+		(size 0.6)
+		(drill 0.3)
+		(layers "F.Cu" "B.Cu")
+		(free yes)
 		(net 2)
 	)
-	(segment
-		(start 53.28 -57.98)
-		(end 54.4573 -56.8027)
-		(width 0.2)
-		(layer "F.Cu")
+	(via
+		(at 28.5 -54.5)
+		(size 0.6)
+		(drill 0.3)
+		(layers "F.Cu" "B.Cu")
+		(free yes)
 		(net 2)
 	)
@@
 		(net 25)
 	)
+	(zone
+		(net 2)
+		(net_name "GND")
+		(layer "F.Cu")
+		(hatch edge 0.5)
+		(priority 1)
+		(connect_pads
+			(clearance 0.5)
+		)
+		(min_thickness 0.25)
+		(filled_areas_thickness no)
+		(fill yes
+			(thermal_gap 0.5)
+			(thermal_bridge_width 0.5)
+		)
+		(polygon
+			(pts
+				(xy -18.5 -78.5) (xy 15 -82.5) (xy 85 -78.5) (xy 76.5 18) (xy -33 8.5) (xy -18 -78.5)
+			)
+		)
+	)
+	(zone
+		(net 2)
+		(net_name "GND")
+		(layer "B.Cu")
+		(hatch edge 0.5)
+		(connect_pads
+			(clearance 0.5)
+		)
+		(min_thickness 0.25)
+		(filled_areas_thickness no)
+		(fill yes
+			(thermal_gap 0.5)
+			(thermal_bridge_width 0.5)
+		)
+		(polygon
+			(pts
+				(xy -10.5 -78.5) (xy 67 -78.5) (xy 66.5 17) (xy -21 16.5) (xy -25 -53)
+			)
+		)
+	)
 	(embedded_fonts no)

Commit message: Add initial KiCad project file for Freezepad PCB design
- Created freezepad-pcb.kicad_pro with default design settings
- Configured design rules, dimensions, and layer settings
- Established net settings and IPC2581 metadata
- Included teardrop and tuning pattern settings for enhanced routing
Parts:
- added REF**: MountingHole_3.2mm_M3_DIN965_Pad_TopBottom, MountingHole:MountingHole_3.2mm_M3_DIN965_Pad_TopBottom, F.Cu at (9.00, -59.5)
- added REF**: MountingHole_3.2mm_M3_DIN965_Pad_TopBottom, MountingHole:MountingHole_3.2mm_M3_DIN965_Pad_TopBottom, F.Cu at (45.0, -42.5)
- added REF**: MountingHole_3.2mm_M3_DIN965_Pad_TopBottom, MountingHole:MountingHole_3.2mm_M3_DIN965_Pad_TopBottom, F.Cu at (45.0, -8.50)
- added REF**: MountingHole_3.2mm_M3_DIN965_Pad_TopBottom, MountingHole:MountingHole_3.2mm_M3_DIN965_Pad_TopBottom, F.Cu at (9.00, -8.50)
Routing:
- net GND: track 5.50 -> 11.2 mm, vias 2 -> 4
- net matrix_col4_row1: track 72.0 -> 77.2 mm
- net matrix_col1_row1: track 137.5 -> 135.2 mm
- net matrix_col1_row5: track 40.7 -> 39.1 mm
- net matrix_col1_row4: track 68.3 -> 66.9 mm
- net matrix_col1_row3: track 98.2 -> 97.0 mm
- net matrix_col4_row3: track 37.8 -> 36.9 mm
- net matrix_col2_row2: track 76.5 -> 77.3 mm
Other:
- board text added: "Est 02.2026"
- board text added: "FreezePad - By Manny Freeze"
- board text added: "MADE BY ME"
